File: kicad/ExpressForEOS/ExpressForEOS.kicad_sch (KiCad schematic)
At the start: 17 parts, among them J1 Conn_02x17_Counter_Clockwise, U1 74HC4051, U10 74LS08, U11 74LS156, U12 74LS156, U13 74LS373, U14 ICM7218BIPI, U15 MAX150BCPP, U16 LM358, U2 74HC4051, U3 74HC4051, U4 74HC4051, U5 CD4066BE, U6 74LS138, U7 74LS374, U8 74LS374, U9 74LS245

Commit message: Schem update
Connections:
- net at U11.13 (A0), U12.13 (A0): now also J1.28 (Pin_28)
- net U11A2B1: now reaches U10.2, U11.14 (Eb1), U11.2 (Ea2), U6.15 (O0)
- net at J1.8 (Pin_8), U11.3 (A1): now also U12.3 (A1)
- net U8Cp: now reaches U6.9 (O6), U8.11 (Cp)
- net U14W: now reaches U14.8 (_WRITE), U6.12 (O3)
- net U7Cp: now reaches U6.10 (O5), U7.11 (Cp)
- net U15Cs: now reaches U15.13 (_CS), U6.11 (O4)
- net U12A2B1: now reaches U10.1, U12.14 (Eb1), U12.2 (Ea2), U6.14 (O1)
- net U12A2B1: no longer J1.28 (Pin_28)
Other:
- moved on the sheet: J1, U10A

Commit message: Schem update
Connections:
- net P8: now reaches J1.8 (Pin_8), U11.3 (A1), U12.3 (A1)
- net P11: now reaches J1.11 (Pin_11), U6.1 (A0)
- net P23: now reaches J1.23 (Pin_23), U6.2 (A1)
- net P13: now reaches J1.13 (Pin_13), U6.3 (A2)
- net P22: now reaches J1.22 (Pin_22), U6.4 (E1), U9.19 (CE)
- net P19: now reaches J1.19 (Pin_19), U15.6 (_WR/RDY), U9.1 (A->B)
- net P16: now reaches J1.16 (Pin_16), U15.8 (_RD)
- net 24xFDX0 renamed XFD0
- net 24xFDX1 renamed XFD1
- net 24xFDX10 renamed XFD10
- net 24xFDX11 renamed XFD11
- net 24xFDX12 renamed XFD12
- net 24xFDX13 renamed XFD13
- net 24xFDX14 renamed XFD14
- net 24xFDX15 renamed XFD15
- net 24xFDX16 renamed XFD16
- net 24xFDX17 renamed XFD17
- net 24xFDX18 renamed XFD18
- net 24xFDX19 renamed XFD19
- net 24xFDX2 renamed XFD2
- net 24xFDX20 renamed XFD20
- net 24xFDX21 renamed XFD21
- net 24xFDX22 renamed XFD22
- net 24xFDX23 renamed XFD23
- net 24xFDX3 renamed XFD3
- net 24xFDX4 renamed XFD4
- net 24xFDX5 renamed XFD5
- net 24xFDX6 renamed XFD6
- net 24xFDX7 renamed XFD7
- net 24xFDX8 renamed XFD8
- net 24xFDX9 renamed XFD9
- net FDR1 renamed FD1
- net FDR2 renamed FD2
- net KEY_SCAN0 renamed KEY_S0
- net KEY_SCAN1 renamed KEY_S1
- net KEY_SCAN2 renamed KEY_S2
- net KEY_SCAN3 renamed KEY_S3
- net KEY_SCAN4 renamed KEY_S4
- net KEY_SCAN5 renamed KEY_S5
- net KEY_SCAN6 renamed KEY_S6
- net KEY_SCAN7 renamed KEY_S7
- net KEY_SCAN8 renamed KEY_S8
Other:
- moved on the sheet: U10E, U16C

Commit message: Schem update
Connections:
- net at U1.3 (A), U16.3 (+), U2.3 (A)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: no longer U4.3 (A)
- net FADERS_TP0 renamed OFD0
- net FADERS_TP1 renamed OFD1
- net FADERS_TP2 renamed OFD2
- net FADERS_TP3 renamed OFD3
- net FADERS_TP4 renamed OFD4
- net FADERS_TP5 renamed OFD5
- net FADERS_TP6 renamed OFD6
- net FADERS_TP7 renamed OFD7
Other:
- moved on the sheet: U2, U3, U4, U5A, U5B, U5C, U5D
