File: kicad/ExpressForEOS/ExpressForEOS.kicad_sch (KiCad schematic)
At the start: 17 parts, among them J1 Conn_02x17_Counter_Clockwise, U1 74HC4051, U10 74LS08, U11 74LS156, U12 74LS156, U13 74LS373, U14 ICM7218BIPI, U15 MAX150BCPP, U16 LM358, U2 74HC4051, U3 74HC4051, U4 74HC4051, U5 CD4066BE, U6 74LS138, U7 74LS374, U8 74LS374, U9 74LS245

Commit message: Schem update
Connections:
- net at U4.3 (A): now also U1.3 (A), U16.3 (+), U2.3 (A), U3.3 (A)
Changed lines of the file:
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@@
   (junction (at 245.11 110.49) (diameter 0) (color 0 0 0 0)
   )
+  (junction (at 162.56 40.64) (diameter 0) (color 0 0 0 0)
+  )
   (junction (at 231.14 13.97) (diameter 0) (color 0 0 0 0)
   )
@@
     (stroke (width 0) (type default))
   )
+  (wire (pts (xy 162.56 40.64) (xy 196.85 40.64))
+    (stroke (width 0) (type default))
+  )
   (wire (pts (xy 116.84 62.23) (xy 124.46 62.23))
     (stroke (width 0) (type default))
@@
     (stroke (width 0) (type default))
   )
+  (wire (pts (xy 196.85 52.07) (xy 196.85 40.64))
+    (stroke (width 0) (type default))
+  )
